File: production/fufupot-ecad/Fufupot/Power.kicad_sch (KiCad schematic)
At the start: 0 parts

Commit message: Power Source
Andy told me to make a simple connector that that shows the 5V and 48V output.
Parts:
- added J1: Conn_01x03, symbol Connector_Generic:Conn_01x03
Connections:
- new net +48V: J1.2 (Pin_2)
- new net +5V: J1.1 (Pin_1)
- new net GND: J1.3 (Pin_3)
Changed lines of the file:
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@@
 (kicad_sch (version 20230121) (generator eeschema)
   (paper "A4")
+  (wire (pts (xy 58.42 36.83) (xy 58.42 41.91))
+    (stroke (width 0) (type default))
+  )
+  (wire (pts (xy 54.61 34.29) (xy 54.61 39.37))
+    (stroke (width 0) (type default))
+  )
+  (wire (pts (xy 57.15 48.26) (xy 57.15 44.45))
+    (stroke (width 0) (type default))
+  )
+  (wire (pts (xy 57.15 44.45) (xy 52.07 44.45))
+    (stroke (width 0) (type default))
+  )
+  (wire (pts (xy 58.42 41.91) (xy 52.07 41.91))
+    (stroke (width 0) (type default))
+  )
+  (wire (pts (xy 54.61 39.37) (xy 52.07 39.37))
+    (stroke (width 0) (type default))
+  )
+  (symbol (lib_id "power:+5V") (at 54.61 34.29 0) (unit 1)
+    (in_bom yes) (on_board yes) (dnp no) (fields_autoplaced)
+    (property "Reference" "#PWR01" (at 54.61 38.1 0)
+      (effects (font (size 1.27 1.27)) hide)
+    )
+    (property "Value" "+5V" (at 54.61 29.21 0)
+      (effects (font (size 1.27 1.27)))
+    )
+    (property "Footprint" "" (at 54.61 34.29 0)
+      (effects (font (size 1.27 1.27)) hide)
+    )
+    (property "Datasheet" "" (at 54.61 34.29 0)
+      (effects (font (size 1.27 1.27)) hide)
+    )
+    (pin "1")
+    (instances
+      (project "Fufupot"
+        (path "/e8bc21b1-eda8-45a8-be25-55b90339183f/9aa61a69-85f8-4fcb-b123-803352e6223c"
+          (reference "#PWR01") (unit 1)
+        )
+      )
+    )
+  )
+  (symbol (lib_id "Connector_Generic:Conn_01x03") (at 46.99 41.91 0) (mirror y) (unit 1)
+    (in_bom yes) (on_board yes) (dnp no)
+    (property "Reference" "J1" (at 44.45 40.64 0)
+      (effects (font (size 1.27 1.27)) (justify left))
+    )
+    (property "Value" "Conn_01x03" (at 44.45 43.18 0)
+      (effects (font (size 1.27 1.27)) (justify left))
+    )
+    (property "Footprint" "" (at 46.99 41.91 0)
+      (effects (font (size 1.27 1.27)) hide)
+    )
+    (property "Datasheet" "~" (at 46.99 41.91 0)
+      (effects (font (size 1.27 1.27)) hide)
+    )
+    (pin "1")
+    (pin "2")
+    (pin "3")
+    (instances
+      (project "Fufupot"
+        (path "/e8bc21b1-eda8-45a8-be25-55b90339183f/9aa61a69-85f8-4fcb-b123-803352e6223c"
+          (reference "J1") (unit 1)
+        )
+      )
+    )
+  )
+  (symbol (lib_id "power:+48V") (at 58.42 36.83 0) (unit 1)
+    (in_bom yes) (on_board yes) (dnp no) (fields_autoplaced)
+    (property "Reference" "#PWR02" (at 58.42 40.64 0)
+      (effects (font (size 1.27 1.27)) hide)
+    )
+    (property "Value" "+48V" (at 58.42 31.75 0)
+      (effects (font (size 1.27 1.27)))
+    )
+    (property "Footprint" "" (at 58.42 36.83 0)
+      (effects (font (size 1.27 1.27)) hide)
+    )
+    (property "Datasheet" "" (at 58.42 36.83 0)
+      (effects (font (size 1.27 1.27)) hide)
+    )
+    (pin "1")
+    (instances
+      (project "Fufupot"
+        (path "/e8bc21b1-eda8-45a8-be25-55b90339183f/9aa61a69-85f8-4fcb-b123-803352e6223c"
+          (reference "#PWR02") (unit 1)
+        )
+      )
+    )
+  )
+  (symbol (lib_id "power:GND") (at 57.15 48.26 0) (unit 1)
+    (in_bom yes) (on_board yes) (dnp no) (fields_autoplaced)
+    (property "Reference" "#PWR03" (at 57.15 54.61 0)
+      (effects (font (size 1.27 1.27)) hide)
+    )
+    (property "Value" "GND" (at 57.15 53.34 0)
+      (effects (font (size 1.27 1.27)))
+    )
+    (property "Footprint" "" (at 57.15 48.26 0)
+      (effects (font (size 1.27 1.27)) hide)
+    )
+    (property "Datasheet" "" (at 57.15 48.26 0)
+      (effects (font (size 1.27 1.27)) hide)
+    )
+    (pin "1")
+    (instances
+      (project "Fufupot"
+        (path "/e8bc21b1-eda8-45a8-be25-55b90339183f/9aa61a69-85f8-4fcb-b123-803352e6223c"
+          (reference "#PWR03") (unit 1)
+        )
+      )
+    )
+  )
 )
