File: production/fufupot-ecad/Fufupot/Power.kicad_sch (KiCad schematic)
At the start: 9 parts, among them J1 Conn_01x03, U1 LM5165DRC

Commit message: Updates unfinished
Parts:
- removed CSS: 33nF, symbol Device:C
- removed Cin, Cout: 1uF, symbol Device:C
- removed J1: Conn_01x03, symbol Connector_Generic:Conn_01x03
- removed L1: 470uH, symbol Device:L
- removed RILIM: 105kOhm, symbol Device:R
- removed Rfbb: 124kOhm, symbol Device:R
- removed Rfbt: 1.4MOhm, symbol Device:R
- removed U1: LM5165DRC, Package_SON:Texas_S-PVSON-N10_ThermalVias, symbol Regulator_Switching:LM5165
