File: production/fufupot-ecad/Fufupot/Fufupot.kicad_sch (KiCad schematic)
At the start: 2 parts, among them U1 EL2001CN

Commit message: Deleted Test
yea
Parts:
- removed RN1: R_Pack07, symbol Device:R_Pack07
- removed U1: EL2001CN, Package_DIP:DIP-8_W7.62mm, symbol Amplifier_Buffer:EL2001CN
Changed lines of the file:
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@@
 (kicad_sch (version 20230121) (generator eeschema)
   (paper "A4")
-  (junction (at 44.45 39.37) (diameter 0) (color 0 0 0 0)
-  )
-  (junction (at 72.39 39.37) (diameter 0) (color 0 0 0 0)
-  )
-  (wire (pts (xy 72.39 39.37) (xy 72.39 33.02))
-    (stroke (width 0) (type default))
-  )
-  (wire (pts (xy 59.69 67.31) (xy 59.69 55.88))
-    (stroke (width 0) (type default))
-  )
-  (wire (pts (xy 86.36 33.02) (xy 86.36 45.72))
-    (stroke (width 0) (type default))
-  )
-  (wire (pts (xy 58.42 45.72) (xy 67.31 45.72))
-    (stroke (width 0) (type default))
-  )
-  (wire (pts (xy 72.39 39.37) (xy 80.01 39.37))
-    (stroke (width 0) (type default))
-  )
-  (wire (pts (xy 59.69 55.88) (xy 74.93 55.88))
-    (stroke (width 0) (type default))
-  )
-  (wire (pts (xy 72.39 33.02) (xy 81.28 33.02))
-    (stroke (width 0) (type default))
-  )
-  (wire (pts (xy 67.31 33.02) (xy 67.31 45.72))
-    (stroke (width 0) (type default))
-  )
-  (wire (pts (xy 72.39 45.72) (xy 72.39 39.37))
-    (stroke (width 0) (type default))
-  )
-  (wire (pts (xy 74.93 55.88) (xy 74.93 67.31))
-    (stroke (width 0) (type default))
-  )
-  (wire (pts (xy 44.45 39.37) (xy 44.45 33.02))
-    (stroke (width 0) (type default))
-  )
-  (wire (pts (xy 44.45 45.72) (xy 44.45 39.37))
-    (stroke (width 0) (type default))
-  )
-  (wire (pts (xy 95.25 33.02) (xy 95.25 45.72))
-    (stroke (width 0) (type default))
-  )
-  (wire (pts (xy 44.45 33.02) (xy 53.34 33.02))
-    (stroke (width 0) (type default))
-  )
-  (wire (pts (xy 44.45 39.37) (xy 52.07 39.37))
-    (stroke (width 0) (type default))
-  )
-  (wire (pts (xy 86.36 45.72) (xy 95.25 45.72))
-    (stroke (width 0) (type default))
-  )
-  (wire (pts (xy 58.42 33.02) (xy 58.42 45.72))
-    (stroke (width 0) (type default))
-  )
-  (symbol (lib_id "power:+3V3") (at 64.77 59.69 0) (unit 1)
-    (in_bom yes) (on_board yes) (dnp no) (fields_autoplaced)
-    (property "Reference" "#PWR02" (at 64.77 63.5 0)
-      (effects (font (size 1.27 1.27)) hide)
-    )
-    (property "Value" "+3V3" (at 64.77 54.61 0)
-      (effects (font (size 1.27 1.27)))
-    )
-    (property "Footprint" "" (at 64.77 59.69 0)
-      (effects (font (size 1.27 1.27)) hide)
-    )
-    (property "Datasheet" "" (at 64.77 59.69 0)
-      (effects (font (size 1.27 1.27)) hide)
-    )
-    (pin "1")
-    (instances
-      (project "Fufupot"
-        (path "/e8bc21b1-eda8-45a8-be25-55b90339183f"
-          (reference "#PWR02") (unit 1)
-        )
-      )
-    )
-  )
-  (symbol (lib_id "power:GND") (at 64.77 74.93 0) (unit 1)
-    (in_bom yes) (on_board yes) (dnp no) (fields_autoplaced)
-    (property "Reference" "#PWR01" (at 64.77 81.28 0)
-      (effects (font (size 1.27 1.27)) hide)
-    )
-    (property "Value" "GND" (at 64.77 80.01 0)
-      (effects (font (size 1.27 1.27)))
-    )
-    (property "Footprint" "" (at 64.77 74.93 0)
-      (effects (font (size 1.27 1.27)) hide)
-    )
-    (property "Datasheet" "" (at 64.77 74.93 0)
-      (effects (font (size 1.27 1.27)) hide)
-    )
-    (pin "1")
-    (instances
-      (project "Fufupot"
-        (path "/e8bc21b1-eda8-45a8-be25-55b90339183f"
-          (reference "#PWR01") (unit 1)
-        )
-      )
-    )
-  )
-  (symbol (lib_id "Device:R_Pack07") (at 43.18 72.39 0) (unit 1)
-    (in_bom yes) (on_board yes) (dnp no) (fields_autoplaced)
-    (property "Reference" "RN1" (at 33.02 71.12 0)
-      (effects (font (size 1.27 1.27)) (justify right))
-    )
-    (property "Value" "R_Pack07" (at 33.02 73.66 0)
-      (effects (font (size 1.27 1.27)) (justify right))
-    )
-    (property "Footprint" "" (at 55.245 72.39 90)
-      (effects (font (size 1.27 1.27)) hide)
-    )
-    (property "Datasheet" "~" (at 43.18 72.39 0)
-      (effects (font (size 1.27 1.27)) hide)
-    )
-    (pin "1")
-    (pin "10")
-    (pin "11")
-    (pin "12")
-    (pin "13")
-    (pin "14")
-    (pin "2")
-    (pin "3")
-    (pin "4")
-    (pin "5")
-    (pin "6")
-    (pin "7")
-    (pin "8")
-    (pin "9")
-    (instances
-      (project "Fufupot"
-        (path "/e8bc21b1-eda8-45a8-be25-55b90339183f"
-          (reference "RN1") (unit 1)
-        )
-      )
-    )
-  )
-  (symbol (lib_id "Amplifier_Buffer:EL2001CN") (at 67.31 67.31 0) (unit 1)
-    (in_bom yes) (on_board yes) (dnp no) (fields_autoplaced)
-    (property "Reference" "U1" (at 78.74 63.1191 0)
-      (effects (font (size 1.27 1.27)))
-    )
-    (property "Value" "EL2001CN" (at 78.74 65.6591 0)
-      (effects (font (size 1.27 1.27)))
-    )
-    (property "Footprint" "Package_DIP:DIP-8_W7.62mm" (at 67.31 76.2 0)
-      (effects (font (size 1.27 1.27)) hide)
-    )
-    (property "Datasheet" "http://www.datasheetlib.com/datasheet/677973/el2001_intersil.html#datasheet" (at 67.31 67.31 0)
-      (effects (font (size 1.27 1.27)) hide)
-    )
-    (pin "1")
-    (pin "2")
-    (pin "3")
-    (pin "4")
-    (pin "5")
-    (pin "6")
-    (pin "7")
-    (pin "8")
-    (instances
-      (project "Fufupot"
-        (path "/e8bc21b1-eda8-45a8-be25-55b90339183f"
-          (reference "U1") (unit 1)
-        )
-      )
-    )
-  )
   (sheet_instances
     (path "/" (page "1"))

Commit message: Made hierarchical schematic sheets
Now everyone can make their changes on separate schematic sheets and no one will have conflicts <3
Other:
- added sheet Fault Protection (FaultProtection.kicad_sch)
- added sheet Heating Circuit (HeatingCircuit.kicad_sch)
- added sheet Motor Driver (MotorDriver.kicad_sch)
- added sheet Power (Power.kicad_sch)
- added sheet User Interface (UI.kicad_sch)
Changed lines of the file:
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@@
 (kicad_sch (version 20230121) (generator eeschema)
   (paper "A4")
+  (sheet (at 118.11 123.19) (size 57.15 20.32) (fields_autoplaced)
+    (stroke (width 0.1524) (type solid))
+    (fill (color 0 0 0 0.0000))
+    (property "Sheetname" "User Interface" (at 118.11 120.6134 0)
+      (effects (font (size 5 5) bold) (justify left bottom))
+    )
+    (property "Sheetfile" "UI.kicad_sch" (at 118.11 144.3866 0)
+      (effects (font (size 2 2)) (justify left top))
+    )
+    (instances
+      (project "Fufupot"
+        (path "/e8bc21b1-eda8-45a8-be25-55b90339183f" (page "5"))
+      )
+    )
+  )
+  (sheet (at 116.84 76.2) (size 59.69 21.59) (fields_autoplaced)
+    (stroke (width 0.1524) (type solid))
+    (fill (color 0 0 0 0.0000))
+    (property "Sheetname" "Heating Circuit" (at 116.84 73.6234 0)
+      (effects (font (size 5 5) bold) (justify left bottom))
+    )
+    (property "Sheetfile" "HeatingCircuit.kicad_sch" (at 116.84 98.6666 0)
+      (effects (font (size 2 2)) (justify left top))
+    )
+    (instances
+      (project "Fufupot"
+        (path "/e8bc21b1-eda8-45a8-be25-55b90339183f" (page "3"))
+      )
+    )
+  )
+  (sheet (at 207.01 76.2) (size 49.53 22.86) (fields_autoplaced)
+    (stroke (width 0.1524) (type solid))
+    (fill (color 0 0 0 0.0000))
+    (property "Sheetname" "Fault Protection" (at 207.01 73.6234 0)
+      (effects (font (size 5 5) bold) (justify left bottom))
+    )
+    (property "Sheetfile" "FaultProtection.kicad_sch" (at 207.01 99.9366 0)
+      (effects (font (size 2 2)) (justify left top))
+    )
+    (instances
+      (project "Fufupot"
+        (path "/e8bc21b1-eda8-45a8-be25-55b90339183f" (page "6"))
+      )
+    )
+  )
+  (sheet (at 125.73 30.48) (size 34.29 21.59) (fields_autoplaced)
+    (stroke (width 0.1524) (type solid))
+    (fill (color 0 0 0 0.0000))
+    (property "Sheetname" "Power" (at 125.73 27.9034 0)
+      (effects (font (size 5 5) bold) (justify left bottom))
+    )
+    (property "Sheetfile" "Power.kicad_sch" (at 125.73 52.9466 0)
+      (effects (font (size 2 2)) (justify left top))
+    )
+    (instances
+      (project "Fufupot"
+        (path "/e8bc21b1-eda8-45a8-be25-55b90339183f" (page "4"))
+      )
+    )
+  )
+  (sheet (at 41.91 77.47) (size 49.53 20.32)
+    (stroke (width 0.1524) (type solid))
+    (fill (color 0 0 0 0.0000))
+    (property "Sheetname" "Motor Driver" (at 41.91 74.93 0)
+      (effects (font (size 5 5) bold) (justify left bottom))
+    )
+    (property "Sheetfile" "MotorDriver.kicad_sch" (at 41.91 98.3746 0)
+      (effects (font (size 2 2)) (justify left top))
+    )
+    (instances
+      (project "Fufupot"
+        (path "/e8bc21b1-eda8-45a8-be25-55b90339183f" (page "2"))
+      )
+    )
+  )
   (sheet_instances
     (path "/" (page "1"))

Commit message: One Page
compiled all edits into one page
Parts:
- added 102PS1J, 102PS1J1, R9: 1k, symbol Device:R
- added 16MHz1: Crystal, 16 MHz Xtal Osc:XTAL_ABL-16_ABR, symbol Device:Crystal
- added BZ1: Buzzer, symbol Device:Buzzer
- added C1: 100n, Capacitor_SMD:C_0805_2012Metric, symbol Device:C_Small
- added C1: 3.3 uF 275V, symbol Device:C_Polarized
- added C1, C2: 22pF, 22 pF Cap:CAP_K-SERIES_15-L2_VIS, symbol Device:C
- added C3: 10uF 25V, symbol Device:C_Polarized
- added C3: 10uF, 10 uF Cap:CAP_YX_5X11_RUB, symbol Device:C_Polarized
- added C4: 0.1uF 63V, symbol Device:C_Polarized
- added C5: 0.37uF 1200V, symbol Device:C_Polarized
- added C5: 0.1 uF, symbol Device:C
- added CSS: 33nF, symbol Device:C
- added Cin, Cout: 1uF, symbol Device:C
- added D1: LED, symbol Device:LED
- added F1: 500mA, Fuse:Fuse_1210_3225Metric, symbol Device:Fuse
- added IC1: FOD3150, DIP762W56P254L966H508Q8N, symbol FOD3150:FOD3150
- added J1: USB_B, Connector_USB:USB_Micro-B_Amphenol_10104110_Horizontal, symbol Connector:USB_B
- added J1: Conn_01x03, symbol Connector_Generic:Conn_01x03
- added J2: Conn_01x04_Pin, symbol Connector:Conn_01x04_Pin
- added J3: Conn_01x05_Pin, symbol Connector:Conn_01x05_Pin
- added J4: Conn_01x03_Pin, symbol Connector:Conn_01x03_Pin
- added L1: L, symbol Device:L
- added L1: 470uH, symbol Device:L
- added L2: 10uH, symbol Device:L
- added R1: 0.1 5W, symbol Device:R
- added R1: 220, symbol Device:R
- added R2: 3.3k, symbol Device:R
- added R2, R5: 330, symbol Device:R
- added R3, R6, R7: 10k, symbol Device:R
- added R3: 10k, Resistor_SMD:R_0805_2012Metric, symbol Device:R_Small
- added R4: 16, symbol Device:R
- added R5, R6, R7, R9: 1k, Resistor_SMD:R_0805_2012Metric, symbol Device:R_Small
- added RILIM: 105kOhm, symbol Device:R
- added Rfbb: 124kOhm, symbol Device:R
- added Rfbt: 1.4MOhm, symbol Device:R
- added SW1: SW_Push, Button_Switch_SMD:SW_DIP_SPSTx04_Slide_6.7x11.72mm_W6.73mm_P2.54mm_LowProfile_JPin, symbol Switch:SW_Push
- added SW2: SW_Push, symbol Switch:SW_Push
- added U1: LM5165DRC, Package_SON:Texas_S-PVSON-N10_ThermalVias, symbol Regulator_Switching:LM5165
- added U1: STGP8NC60KD, TO-220FP_STM, symbol STGP8NC60KD:STGP8NC60KD
- added U2: FT232RL, Package_SO:SSOP-28_5.3x10.2mm_P0.65mm, symbol Interface_USB:FT232RL
- added U2: ATMEGA328P-PN, footprints:28P3_ATM, symbol 2023-10-12_03-24-27:ATMEGA328P-PN
- added U3: USBLC6-2SC6, Package_TO_SOT_SMD:SOT-23-6, symbol Power_Protection:USBLC6-2SC6
Connections:
- new net: C3.2, IC1.5 (VSS), R1.1, R2.1, R3.1, R3.2, R4.2, U1.1 (G), U1.3 (E)
- new net: R7.1, U2.1 (TXD)
- new net: L1.1, U1.1 (SW)
- new net: RILIM.1, U1.3 (ILIM)
- new net: CSS.1, U1.4 (SS)
- new net: Rfbb.1, Rfbt.2, U1.8 (FB)
- new net: C5.2, L1.2, U1.2 (C)
- new net: C1.1, C5.1, L1.1, L2.2
- new net: R3.2, U2.19 (~{RESET})
- new net: R6.1, U2.5 (RXD)
- new net: IC1.6 (VO1), IC1.7 (VO2), R4.1
- new net: 16MHz1.1, C2.2, U2.10 (PB7)
- new net: D1.2 (A), R1.2
- new net: IC1.2 (ANODE), R5.2
- new net: 16MHz1.2, C1.2, U2.9 (PB6)
- new net: F1.1, J1.1 (VBUS)
- new net +15V: C3.1, IC1.8 (VDD)
- new net +3V3: C1.1, U2.17 (3V3OUT)
- new net +48V: BZ1.2 (+), C1.1, C1.2, C1.2, C2.1, C3.2, C4.2, C5.2, CSS.2, Cin.1, Cin.2, Cout.1, Cout.2, D1.1 (K), IC1.3 (CATHODE), J1.2 (Pin_2), J1.3 (Pin_3), J1.4 (GND), J4.1 (Pin_1), J4.3 (Pin_3), L1.2, L2.1, R1.2, R5.1, R6.1, R7.1, RILIM.2, Rfbb.2, Rfbt.1, SW1.1, SW2.1, U1.10 (GND), U1.11 (PAD), U1.2 (VIN), U1.5 (RT), U1.7 (EN), U2.18 (GND), U2.21 (GND), U2.22 (GND), U2.25 (AGND), U2.26 (TEST), U2.7 (GND), U2.8 (GND), U3.2 (GND)
- new net +5V: 102PS1J.2, 102PS1J1.2, C3.1, C5.1, J1.1 (Pin_1), J4.2 (Pin_2), R3.1, U2.20 (AVCC), U2.20 (VCC), U2.4 (VCCIO), U2.7 (VCC)
- new net A1: C4.1, J3.5 (Pin_5), R2.2, U2.24 (PC1)
- new net A2: 102PS1J.1, J3.4 (Pin_4), R6.2, U2.25 (PC2)
- new net A3: 102PS1J1.1, J3.3 (Pin_3), R7.2, U2.26 (PC3)
- new net A4: J3.2 (Pin_2), U2.27 (PC4)
- new net A5: J3.1 (Pin_1), U2.28 (PC5)
- new net D1: BZ1.1 (-)
- new net D2: R1.1
- new net D3: R2.1
- new net D9: R5.1
- new net DTR: R5.2, R9.1, SW1.2, U2.2 (DTR)
- new net Heat: U2.23 (PC0)
- new net LED_SGN: R2.2
- new net MISO: J2.2 (Pin_2), U2.18 (PB4)
- new net MOSI: J2.3 (Pin_3), U2.17 (PB3)
- new net PWM Speed Control: U2.15 (PB1)
- new net RESET: R9.2, SW2.2, U2.1 (PC6)
- new net RX: R6.2, U2.2 (PD0)
- new net SCK: J2.1 (Pin_1), U2.19 (PB5)
- new net SS: J2.4 (Pin_4), U2.16 (PB2)
- new net TX: R7.2, U2.3 (PD1)
- new net USB_CON_D+: J1.3 (D+), U3.1 (I/O1)
- new net USB_CON_D-: J1.2 (D-), U3.3 (I/O2)
- new net USB_D+: U2.15 (USBD+), U3.6 (I/O1)
- new net USB_D-: U2.16 (USBD-), U3.4 (I/O2)
- new net VBUS: F1.2, U3.5 (VBUS)
- new net VCC: R9.1, R9.2
- no-connect marks 0 -> 23
Other:
- removed sheet Fault Protection
- removed sheet Heating Circuit
- removed sheet Motor Driver
- removed sheet Power
- removed sheet User Interface
- note added: "Buck Converter: 48V -> 15V"
- note added: "Connects with Heating Schematic"
- note added: "Inductive Heating"
- note added: "Microcontroller"
- note added: "Motor Driver PCB Screw Terminal"
- note added: "Power: 48V, 5V"
- note added: "Reset Button for MCU"
- note added: "SPI Bus Headers and GPIO Pins"
- note added: "Temperature Sensing"
- note added: "This connects to the 0-5V terminal on the motor controller"
- note added: "USB CONN AND PROTECTION"
- note added: "USB-UART BRIDGE"
- note added: "User Interface"
- company: (none) -> Generate
- title: (none) -> Fufu Pot Schematic

Commit message: Labels
Added GUI labels
Parts:
- removed J3: Conn_01x05_Pin, symbol Connector:Conn_01x05_Pin
- added J1: Conn_01x02_Pin, symbol Connector:Conn_01x02_Pin
- renumbered 102PS1J to 102PS1J2, 102PS1J1 to 102PS1J3, 16MHz1 to 16MHz2, C1 to C10, C2 to C11, C3 to C12, C5 to C13, CSS to CSS1, Cin to Cin1, Cout to Cout1, J1 to J5, J2 to J7, J4 to J9, L1 to L3, R6 to R10, R7 to R11, R9 to R3, RILIM to RILIM1, Rfbb to Rfbb1, Rfbt to Rfbt1, SW2 to SW3, U1 to U5, U2 to U7
Connections:
- net A1: now also U7.27 (PC4); no longer U7.24 (PC1)
- net A2: now also U7.28 (PC5); no longer U7.25 (PC2)
- net A4: now also U7.23 (PC0), J1.1 (Pin_1); no longer U7.27 (PC4)
- net A5: now also U7.24 (PC1), J1.2 (Pin_2); no longer U7.28 (PC5)
- net Heat: now also U7.5 (PD3); no longer U7.23 (PC0)
- net D_Blue: now reaches U7.11 (PD5)
- net D_LEDStrip: now reaches U7.12 (PD6)
- net D_Buzz: now reaches U7.13 (PD7)
- net D_Switch: now reaches U7.14 (PB0)
- net D_LED: now reaches U7.4 (PD2)
- net D_Red: now reaches U7.6 (PD4)
- new net D_Green: U7.25 (PC2)
- no-connect marks 23 -> 16

Commit message: Updated Buck Converter
Modified buck converter values and reference designators
Parts:
- C3: renamed from Cout1; value 1uF -> 10uF
- L1: renamed from L3; value 470uH -> 47uH
- R1: renamed from Rfbt1; value 1.4MOhm -> 900kOhm
- R2: renamed from Rfbb1; value 124kOhm -> 80kOhm
- renumbered Cin1 to C1, CSS1 to C2, RILIM1 to R3, U5 to U1
Connections:
- net +48V is gone; now on net +15V: BZ1.2 (+), C1.1, C1.2, C1.2, C1.2, C10.1, C11.1, C12.2, C13.2, C2.2, C3.1, C3.2, C4.2, D1.1 (K), IC1.3 (CATHODE), J1.4 (GND), J5.2 (Pin_2), J5.3 (Pin_3), J9.1 (Pin_1), J9.3 (Pin_3), L1.2, L2.1, R1.1, R1.2, R10.1, R11.1, R2.2, R3.2, R5.1, SW1.1, SW3.1, U1.10 (GND), U1.11 (PAD), U1.2 (VIN), U1.5 (RT), U1.7 (EN), U2.18 (GND), U2.21 (GND), U2.25 (AGND), U2.26 (TEST), U2.7 (GND), U3.2 (GND), U7.22 (GND), U7.8 (GND)
- net D1 is gone; now on net D_Buzz: BZ1.1 (-)
- net D2 is gone; now on net D_LED: R1.1
- net D3 is gone; now on net D_LEDStrip: R2.1
- net D_Blue is gone; now on net Blue_LED: U7.11 (PD5)
- net Heat is gone; now on net D9: U7.5 (PD3)
Other:
- note added: "A1-3 & D9 Connects with Heating Schematic"
- note added: "A4 & A5 extra gpio"
- note added: "PWM_S_C connects to the 0-5V terminal on the motor controller"
- note removed: "Connects with Heating Schematic"
- note removed: "This connects to the 0-5V terminal on the motor controller"

Commit message: finished schem
Parts:
- removed 16MHz2: Crystal, 16 MHz Xtal Osc:XTAL_ABL-16_ABR, symbol Device:Crystal
- removed BZ1: Buzzer, symbol Device:Buzzer
- removed C10: 22pF, 22 pF Cap:CAP_K-SERIES_15-L2_VIS, symbol Device:C
- removed C12: 10uF, 10 uF Cap:CAP_YX_5X11_RUB, symbol Device:C_Polarized
- removed C13: 0.1 uF, symbol Device:C
- removed D1: LED, symbol Device:LED
- removed R1: 220, symbol Device:R
- removed R2: 330, symbol Device:R
- removed U7: ATMEGA328P-PN, footprints:28P3_ATM, symbol 2023-10-12_03-24-27:ATMEGA328P-PN
- added 16MHz1: Crystal, 16 MHz Xtal Osc:XTAL_ABL-16_ABR, symbol Device:Crystal
- added C10: 10uF, 10 uF Cap:CAP_YX_5X11_RUB, symbol Device:C_Polarized
- added C4, C5: 22pF, 22 pF Cap:CAP_K-SERIES_15-L2_VIS, symbol Device:C
- added J2, J4: Conn_01x02_Pin, symbol Connector:Conn_01x02_Pin
- added J3: Conn_01x03_Pin, symbol Connector:Conn_01x03_Pin
- added J8: Conn_01x04_Pin, symbol Connector:Conn_01x04_Pin
- added R2: 330, symbol Device:R
- added R2: 220, symbol Device:R
- added R4, R5: 0, symbol Device:R
- added U2: ATMEGA328P-PN, footprints:28P3_ATM, symbol 2023-10-12_03-24-27:ATMEGA328P-PN
- C11: value 22pF -> 0.1 uF; footprint 22 pF Cap:CAP_K-SERIES_15-L2_VIS -> (none)
Connections:
- net +15V: now also C11.2, C10.2, C4.1, C5.1, J2.1 (Pin_1), J3.3 (Pin_3), J4.1 (Pin_1), J8.1 (Pin_1), J8.4 (Pin_4), R4.2, R5.2, U2.22 (GND), U2.8 (GND); no longer C11.1
- net +5V: now also C11.1, C10.1, J3.2 (Pin_2), U2.20 (AVCC), U2.7 (VCC)
- net A1: now also U2.27 (PC4)
- net A2: now also U2.28 (PC5)
- net A3: now also U2.26 (PC3)
- net A4: now also U2.23 (PC0)
- net A5: now also U2.24 (PC1)
- net D9: now also U2.5 (PD3)
- net D_Buzz: now also J4.2 (Pin_2), U2.13 (PD7)
- net D_LED: now also R2.1, U2.4 (PD2)
- net D_LEDStrip: now also R2.1, U2.11 (PD5)
- net D_Red: now also J8.2 (Pin_2), U2.6 (PD4)
- net D_Switch: now also J8.3 (Pin_3), U2.14 (PB0)
- net MISO: now also U2.18 (PB4)
- net MOSI: now also U2.17 (PB3)
- net PWM Speed Control: now also U2.15 (PB1)
- net RESET: now also U2.1 (PC6)
- net RX: now also U2.2 (PD0)
- net SCK: now also U2.19 (PB5)
- net SS: now also U2.16 (PB2)
- net TX: now also U2.3 (PD1)
- new net: 16MHz1.1, C5.2, U2.10 (PB7)
- new net: J3.1 (Pin_1), R2.2
- new net: R4.1, U2.25 (PC2)
- new net: 16MHz1.2, C4.2, U2.9 (PB6)
- new net: J2.2 (Pin_2), R2.2

Commit message: Updates unfinished
Parts:
- removed J9: Conn_01x03_Pin, symbol Connector:Conn_01x03_Pin
- removed R5: 0, symbol Device:R
- added J10: Conn_01x03, symbol Connector_Generic:Conn_01x03
- added R20: 0, symbol Device:R
- C1: footprint (none) -> ECQUAAF335LD; symbol Device:C_Polarized -> ECQUAAF335LD:ECQUAAF335LD; Height (none) -> 30.5; Manufacturer_Name (none) -> Panasonic; Manufacturer_Part_Number (none) -> ECQUAAF335LD
- renumbered 102PS1J2 to 102PS1J1, 102PS1J3 to 102PS1J2, C2 to C3, C3 to C4, C4 to C5, C5 to C6, C10 to C7, C11 to C8, J7 to J1, J5 to J3, J1 to J4, J2 to J5, J3 to J6, J4 to J7, J8 to J9, R10 to R12, R11 to R13, R4 to R19, R1 to R5, R2 to R6, R3 to R7, SW3 to SW1, U1 to U2, U2 to U4
Connections:
- net +15V: no longer C1.1, C1.2, C1.2, C1.2, C3.2, C4.2, C4.2, C5.1, C6.1, C7.2, C8.2, IC1.3 (CATHODE), J1.4 (GND), J3.2 (Pin_2), J3.3 (Pin_3), J5.1 (Pin_1), J6.3 (Pin_3), J7.1 (Pin_1), J9.1 (Pin_1), J9.4 (Pin_4), L2.1, R1.2, R12.1, R13.1, R19.2, R3.2, R5.1, R6.2, SW1.1, SW1.1, U2.10 (GND), U2.11 (PAD), U2.18 (GND), U2.2 (VIN), U2.21 (GND), U2.25 (AGND), U2.26 (TEST), U2.5 (RT), U2.7 (EN), U2.7 (GND), U3.2 (GND), U4.22 (GND), U4.8 (GND)
- net at U4.12 (PD6): now also R20.1
- new net +48V: C1.1, J3.2 (Pin_2), L2.1, U2.2 (VIN), U2.7 (EN)
- new net GND: C1.2, C1.2, C3.2, C4.2, C4.2, C5.1, C6.1, C7.2, C8.2, IC1.3 (CATHODE), J1.4 (GND), J3.3 (Pin_3), J5.1 (Pin_1), J6.3 (Pin_3), J7.1 (Pin_1), J9.1 (Pin_1), J9.4 (Pin_4), R1.2, R12.1, R13.1, R19.2, R20.2, R3.2, R5.1, R6.2, SW1.1, SW1.1, U2.10 (GND), U2.11 (PAD), U2.18 (GND), U2.21 (GND), U2.25 (AGND), U2.26 (TEST), U2.5 (RT), U2.7 (GND), U3.2 (GND), U4.22 (GND), U4.8 (GND)
- no-connect marks 16 -> 18
Other:
- note added: "48V Source"
