File: production/fufupot-ecad/Fufupot/Fufupot.kicad_pcb (KiCad board)
At the start: 4 copper layers, 116.8 x 124.5 mm, 56 parts, among them IC1 FOD3150, J1 Conn_01x04, J10 Conn_01x03, J11 Conn_01x03, J12 Conn_01x02, J13 Conn_01x03, J2 USB_B, J3 Conn_01x03, J4 Conn_01x02, J6 Conn_01x02, J7 Conn_01x02, J8 Conn_01x04, J9 Conn_01x02, SW1 SW_Push, SW2 SW_Push, U1 USBLC6-2SC6, U2 LM5165DRC, U3 FT232RL, U4 ATMEGA328P-PN, U5 STGP8NC60KD

Commit message: Everything Fixed
Parts:
- U2: footprint Package_SON:Texas_S-PVSON-N10_ThermalVias -> BuckConverter:DRC0010J
- moved J2 10.2 mm to (142.2, 133.7), turned to 0 degrees
- moved R17 7.62 mm to (152.4, 94.0)
Routing:
- net Net-(IC1-VSS): track 98.4 -> 85.5 mm
- net USB_CON_D-: track 6.40 -> 13.6 mm
- net Net-(J2-VBUS): track 8.71 -> 15.9 mm
- net USB_CON_D+: track 11.4 -> 13.6 mm
- net GND: track 76.2 -> 74.1 mm
Other:
- board text added: "FuFu Pot Katie Dewhurst Luis Rodriguez Elise Cooke Cat Menten Version 1"
- board text removed: "FuFu Pot Katie Dewhurst Elise Cooke Luis Rodriguez Cat Menten Version 1"

Commit message: Version 3
Parts:
- added TP3: TestPoint, TestPoint:TestPoint_Pad_2.0x2.0mm, F.Cu at (129.5, 101.6)
- moved U1 2.81 mm to (128.4, 134.6)
Routing:
- net Net-(J4-Pin_2): track 0.00 -> 56.5 mm
- net Net-(J4-Pin_1): track 0.00 -> 30.0 mm
- net +16V: track 18.1 -> 30.0 mm
- net GND: track 74.1 -> 77.4 mm
- net USB_D-: track 2.61 -> 5.55 mm
- net USB_D+: track 2.98 -> 5.79 mm
- net USB_CON_D-: track 13.6 -> 10.8 mm
- net USB_CON_D+: track 13.6 -> 10.8 mm
- removed copper zone on F.Cu, net (none)
