File: production/fufupot-ecad/Fufupot/Andy File/Fufupot.kicad_pcb (KiCad board)
At the start: 4 copper layers, 116.8 x 124.5 mm, 56 parts, among them IC1 FOD3150, J1 Conn_01x04, J10 Conn_01x03, J11 Conn_01x03, J12 Conn_01x02, J13 Conn_01x03, J2 USB_B, J3 Conn_01x03, J4 Conn_01x02, J6 Conn_01x02, J7 Conn_01x02, J8 Conn_01x04, J9 Conn_01x02, SW1 SW_Push, SW2 SW_Push, U1 USBLC6-2SC6, U2 LM5165DRC, U3 FT232RL, U4 ATMEGA328P-PN, U5 STGP8NC60KD

Commit message: Fix some errors
Routing:
- net Net-(J4-Pin_2): track 0.00 -> 51.3 mm
- net Net-(J4-Pin_1): track 0.00 -> 33.3 mm
- net GND: track 76.2 -> 90.5 mm, vias 29 -> 33
- net +5V: track 52.4 -> 66.2 mm, vias 9 -> 10
Other:
- board text removed: "FuFu Pot Katie Dewhurst Elise Cooke Luis Rodriguez Cat Menten Version 1"
Changed lines of the file:
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@@
   (gr_rect (start 50.8 40.64) (end 167.64 165.1)
     (stroke (width 0.2) (type default)) (fill none) (layer "Edge.Cuts"))
-  (gr_text "FuFu Pot \nKatie Dewhurst\nElise Cooke\nLuis Rodriguez\nCat Menten\nVersion 1\n" (at 147.32 63.5) (layer "Dwgs.User")
-    (effects (font (size 1 1) (thickness 0.15)) (justify left bottom))
-  )
   (segment (start 120.346776 133.169415) (end 120.637156 133.459795) (width 0.25) (layer "F.Cu") (net 1))
   (segment (start 120.637156 133.459795) (end 120.637156 138.386571) (width 0.25) (layer "F.Cu") (net 1))
@@
   (segment (start 92.999415 103.159415) (end 90.725 103.159415) (width 0.25) (layer "F.Cu") (net 6))
   (segment (start 104.14 106.68) (end 109.22 106.68) (width 0.25) (layer "F.Cu") (net 6))
+  (segment (start 83.82 123.479415) (end 81.28 120.939415) (width 0.25) (layer "F.Cu") (net 6))
   (segment (start 107.395 120.224415) (end 109.22 118.399415) (width 0.25) (layer "F.Cu") (net 6))
+  (segment (start 68.58 124.46) (end 68.58 121.92) (width 0.25) (layer "F.Cu") (net 6))
   (segment (start 109.529415 106.989415) (end 111.235 106.989415) (width 0.25) (layer "F.Cu") (net 6))
   (segment (start 68.58 114.3) (end 66.04 111.76) (width 0.25) (layer "F.Cu") (net 6))
   (segment (start 91.44 123.479415) (end 88.9 123.479415) (width 0.25) (layer "F.Cu") (net 6))
+  (segment (start 81.28 120.939415) (end 81.28 118.399415) (width 0.25) (layer "F.Cu") (net 6))
   (segment (start 96.52 106.68) (end 92.999415 103.159415) (width 0.25) (layer "F.Cu") (net 6))
   (segment (start 116.25 127.969415) (end 114.72 127.969415) (width 0.25) (layer "F.Cu") (net 6))
@@
   (segment (start 71.12 104.14) (end 68.58 106.68) (width 0.25) (layer "F.Cu") (net 6))
   (segment (start 117.555 140.544415) (end 116.84 141.259415) (width 0.25) (layer "F.Cu") (net 6))
+  (segment (start 88.9 123.479415) (end 83.82 123.479415) (width 0.25) (layer "F.Cu") (net 6))
   (segment (start 117.555 138.719415) (end 117.555 140.544415) (width 0.25) (layer "F.Cu") (net 6))
   (segment (start 107.395 120.939415) (end 107.395 120.224415) (width 0.25) (layer "F.Cu") (net 6))
   (segment (start 71.12 96.52) (end 71.12 104.14) (width 0.25) (layer "F.Cu") (net 6))
+  (via (at 68.58 121.92) (size 0.8) (drill 0.4) (layers "F.Cu" "B.Cu") (free) (net 6))
   (via (at 116.84 128.559415) (size 0.8) (drill 0.4) (layers "F.Cu" "B.Cu") (free) (net 6))
   (via (at 68.58 106.68) (size 0.8) (drill 0.4) (layers "F.Cu" "B.Cu") (free) (net 6))
@@
   (segment (start 109.22 101.6) (end 106.68 101.6) (width 0.25) (layer "F.Cu") (net 35))
   (segment (start 116.655 95.724415) (end 116.405 95.474415) (width 0.25) (layer "F.Cu") (net 35))
+  (segment (start 101.6 147.32) (end 101.6 149.86) (width 0.25) (layer "F.Cu") (net 35))
+  (segment (start 78.74 118.399415) (end 78.74 120.939415) (width 0.25) (layer "F.Cu") (net 35))
   (segment (start 140.24 95.539415) (end 137.16 95.539415) (width 0.25) (layer "F.Cu") (net 35))
   (segment (start 67.025 144.78) (end 66.5 144.255) (width 0.25) (layer "F.Cu") (net 35))
@@
   (segment (start 119.38 133.499795) (end 119.38 133.639415) (width 0.25) (layer "F.Cu") (net 35))
   (segment (start 126.275 108.239415) (end 125.3625 107.326915) (width 0.25) (layer "F.Cu") (net 35))
+  (segment (start 81.82 123.479415) (end 79.28 120.939415) (width 0.25) (layer "F.Cu") (net 35))
   (segment (start 127.95 134.589415) (end 126.735 134.589415) (width 0.25) (layer "F.Cu") (net 35))
   (segment (start 126.275 108.954415) (end 126.275 108.239415) (width 0.25) (layer "F.Cu") (net 35))
@@
   (segment (start 99.695 123.479415) (end 100.619415 123.479415) (width 0.25) (layer "F.Cu") (net 35))
   (segment (start 79.03 100.909415) (end 78.74 100.619415) (width 0.25) (layer "F.Cu") (net 35))
+  (segment (start 86.36 147.32) (end 86.36 149.86) (width 0.25) (layer "F.Cu") (net 35))
   (segment (start 109.825 97.474415) (end 109.035 98.264415) (width 0.25) (layer "F.Cu") (net 35))
   (segment (start 63.5 116.84) (end 63.5 114.3) (width 0.25) (layer "F.Cu") (net 35))
@@
   (segment (start 127 141.259415) (end 125.41 141.259415) (width 0.25) (layer "F.Cu") (net 35))
   (segment (start 80.57 100.909415) (end 79.03 100.909415) (width 0.25) (layer "F.Cu") (net 35))
+  (segment (start 73.66 124.46) (end 73.66 121.92) (width 0.25) (layer "F.Cu") (net 35))
   (segment (start 103.955 98.264415) (end 103.955 95.724415) (width 0.25) (layer "F.Cu") (net 35))
   (segment (start 91.44 126.019415) (end 88.9 126.019415) (width 0.25) (layer "F.Cu") (net 35))
@@
   (segment (start 119.91 130.569415) (end 121.92 130.569415) (width 0.25) (layer "F.Cu") (net 35))
   (segment (start 109.22 115.859415) (end 105.965 115.859415) (width 0.25) (layer "F.Cu") (net 35))
+  (segment (start 79.28 120.939415) (end 78.74 120.939415) (width 0.25) (layer "F.Cu") (net 35))
+  (via (at 78.74 120.939415) (size 0.8) (drill 0.4) (layers "F.Cu" "B.Cu") (free) (net 35))
   (via (at 109.22 115.859415) (size 0.8) (drill 0.4) (layers "F.Cu" "B.Cu") (free) (net 35))
+  (via (at 101.6 149.86) (size 0.8) (drill 0.4) (layers "F.Cu" "B.Cu") (free) (net 35))
   (via (at 152.4 132.08) (size 0.8) (drill 0.4) (layers "F.Cu" "B.Cu") (free) (net 35))
   (via (at 101.6 124.46) (size 0.8) (drill 0.4) (layers "F.Cu" "B.Cu") (free) (net 35))
@@
   (via (at 121.92 123.479415) (size 0.8) (drill 0.4) (layers "F.Cu" "B.Cu") (net 35))
   (via (at 78.74 100.619415) (size 0.8) (drill 0.4) (layers "F.Cu" "B.Cu") (free) (net 35))
-  (via (at 125.3625 107.326915) (size 0.8) (drill 0.4) (layers "F.Cu" "B.Cu") (free) (net 35))
+  (via micro (at 125.3625 107.326915) (size 0.8) (drill 0.4) (layers "F.Cu" "In1.Cu") (free) (net 35))
   (via (at 106.68 101.6) (size 0.8) (drill 0.4) (layers "F.Cu" "B.Cu") (free) (net 35))
   (via (at 101.415 95.724415) (size 0.8) (drill 0.4) (layers "F.Cu" "B.Cu") (free) (net 35))
@@
   (via (at 116.655 95.724415) (size 0.8) (drill 0.4) (layers "F.Cu" "B.Cu") (free) (net 35))
   (via (at 109.22 127) (size 0.8) (drill 0.4) (layers "F.Cu" "B.Cu") (free) (net 35))
+  (via (at 73.66 121.92) (size 0.8) (drill 0.4) (layers "F.Cu" "B.Cu") (free) (net 35))
   (via (at 132.08 55.88) (size 0.8) (drill 0.4) (layers "F.Cu" "B.Cu") (free) (net 35))
   (via (at 132.08 58.42) (size 0.8) (drill 0.4) (layers "F.Cu" "B.Cu") (free) (net 35))
   (via (at 68.58 144.78) (size 0.8) (drill 0.4) (layers "F.Cu" "B.Cu") (free) (net 35))
   (via (at 83.82 136.179415) (size 0.8) (drill 0.4) (layers "F.Cu" "B.Cu") (free) (net 35))
+  (via (at 86.36 149.86) (size 0.8) (drill 0.4) (layers "F.Cu" "B.Cu") (free) (net 35))
   (via micro (at 125 87.919415) (size 0.8) (drill 0.4) (layers "F.Cu" "In1.Cu") (free) (net 35))
   (segment (start 116.655 100.804415) (end 115.095585 100.804415) (width 0.25) (layer "F.Cu") (net 36))
@@
   (via (at 120.939415 90.459415) (size 0.8) (drill 0.4) (layers "F.Cu" "B.Cu") (free) (net 37))
   (segment (start 120.939415 90.459415) (end 147.86 90.459415) (width 0.25) (layer "B.Cu") (net 37))
+  (segment (start 90.47 61.93) (end 90.47 55.88) (width 0.25) (layer "F.Cu") (net 38))
+  (segment (start 85.23 73.66) (end 85.23 67.17) (width 0.25) (layer "F.Cu") (net 38))
+  (segment (start 71.12 68.84) (end 75.94 73.66) (width 0.25) (layer "F.Cu") (net 38))
+  (segment (start 75.94 73.66) (end 85.23 73.66) (width 0.25) (layer "F.Cu") (net 38))
+  (segment (start 85.23 73.66) (end 85.23 77.61) (width 0.25) (layer "F.Cu") (net 38))
+  (segment (start 90.19 82.57) (end 90.19 86.885) (width 0.25) (layer "F.Cu") (net 38))
+  (segment (start 85.23 67.17) (end 90.47 61.93) (width 0.25) (layer "F.Cu") (net 38))
+  (segment (start 85.23 77.61) (end 90.19 82.57) (width 0.25) (layer "F.Cu") (net 38))
+  (segment (start 103.86 78.74) (end 102.73 77.61) (width 0.25) (layer "F.Cu") (net 39))
+  (segment (start 102.73 77.61) (end 102.73 73.66) (width 0.25) (layer "F.Cu") (net 39))
+  (segment (start 107.634415 87.314415) (end 104.14 83.82) (width 0.25) (layer "F.Cu") (net 39))
+  (segment (start 92.69 86.885) (end 100.835 78.74) (width 0.25) (layer "F.Cu") (net 39))
+  (segment (start 104.14 83.82) (end 104.14 78.74) (width 0.25) (layer "F.Cu") (net 39))
+  (segment (start 104.14 78.74) (end 103.86 78.74) (width 0.25) (layer "F.Cu") (net 39))
+  (segment (start 101.6 78.74) (end 102.73 77.61) (width 0.25) (layer "F.Cu") (net 39))
+  (segment (start 100.835 78.74) (end 101.6 78.74) (width 0.25) (layer "F.Cu") (net 39))
+  (segment (start 111.155 87.314415) (end 107.634415 87.314415) (width 0.25) (layer "F.Cu") (net 39))
   (segment (start 129.365 95.539415) (end 126.825 98.079415) (width 0.25) (layer "F.Cu") (net 40))
   (segment (start 130.08 96.254415) (end 129.365 95.539415) (width 0.25) (layer "F.Cu") (net 40))
@@
       )
     )
-  )
-  (zone (net 0) (net_name "") (layer "F.Cu") (hatch edge 0.5)
-    (priority 16)
-    (connect_pads (clearance 0.5))
-    (min_thickness 0.25) (filled_areas_thickness no)
-    (fill yes (thermal_gap 0.5) (thermal_bridge_width 0.5) (island_removal_mode 1) (island_area_min 10))
-    (polygon
-      (pts
-        (xy 104.14 76.2)
-        (xy 109.22 86.36)
-        (xy 104.14 86.36)
-      )
-    )
